File: hardware/ble_ir_remote.kicad_pcb (KiCad board)
At the start: 2 copper layers, 40.1 x 40 mm, 42 parts, among them J1 TYPE-C-31-M-12, J2 Debug connector, Q1 MMBT3904, U1 ESP32-C3-MINI-1-N4, U2 XC6206PxxxMR, U3 SRV05-4

Commit message: basic placement
Parts:
- C11, C9: value 100n -> 10u
- moved R3 78.9 mm to (171.4, 69.9), turned to -90 degrees
- moved C1 72.4 mm to (167.9, 69.8), turned to 90 degrees
- moved R4 72.3 mm to (170.9, 97.8), turned to -90 degrees
- moved D1 68.9 mm to (145.3, 55.9)
- moved C2 64.6 mm to (167.1, 97.8), turned to 90 degrees
- moved R2 62.9 mm to (144.3, 61.7)
- moved Q1 61.3 mm to (151.9, 63.8), turned to 90 degrees
- moved C3 60.1 mm to (148.1, 84.1), turned to 90 degrees
- moved R1 59.3 mm to (150.1, 68.1)
- moved R9 58.1 mm to (151.9, 98.0), turned to -90 degrees
- moved S1 50.0 mm to (166.4, 64.3)
- moved J1 49.1 mm to (147.3, 141.8)
- moved C11 48.6 mm to (153.4, 106.7), turned to -90 degrees
- moved S6 48.4 mm to (126.7, 78.2)
- moved S5 46.1 mm to (126.7, 91.4)
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Routing:
- net VBUS: track 0.00 -> 21.3 mm, vias 0 -> 2
- net /USB_D+: track 0.00 -> 21.2 mm, vias 0 -> 2
- net /USB_D-: track 0.00 -> 17.5 mm
- net Net-(J1-PadB5): track 0.00 -> 9.83 mm
- net Net-(J1-PadA5): track 0.00 -> 9.23 mm
- net GND: track 0.00 -> 4.11 mm, vias 0 -> 2
- added copper zone on F.Cu, net GND
Other:
- board size 40.1 x 40 mm -> 61 x 90.7 mm

Commit message: routing
Parts:
- moved J2 58.4 mm to (173.9, 123.2)
- moved R2 6.40 mm to (141.7, 55.9)
- moved R14 5.68 mm to (132.7, 120.7)
- moved R1 1.31 mm to (150.9, 69.1), turned to 90 degrees
- moved R12 1.29 mm to (156.5, 140.9), turned to -90 degrees
Connections:
- J2 pad 1: VBUS -> GND
- J2 pad 3: /RST -> /TXD0
- J2 pad 5: /TXD0 -> /BOOT0
- J2 pad 6: /BOOT0 -> /BOOT1
- J2 pad 7: /BOOT1 -> /RST
- J2 pad 8: GND -> VBUS
Routing:
- net +3V3: track 0.00 -> 369.2 mm, vias 0 -> 8
- net /RST: track 0.00 -> 60.1 mm, vias 0 -> 4
- net /BOOT1: track 0.00 -> 55.9 mm, vias 0 -> 2
- net /SW_STANDBY: track 0.00 -> 45.1 mm
- net /BOOT0: track 0.00 -> 42.5 mm, vias 0 -> 2
- net /SW_VOLM: track 0.00 -> 42.3 mm
- net /IR_OUT: track 0.00 -> 36.9 mm
- net VBUS: track 21.3 -> 57.6 mm
- net /SW_PROG2: track 0.00 -> 30.7 mm
- net /RXD0: track 0.00 -> 27.6 mm
- net /SW_BASSM: track 0.00 -> 27.1 mm
- net /TXD0: track 0.00 -> 25.9 mm
- net /SW_VOLP: track 0.00 -> 25.2 mm
- net /SW_BASSP: track 0.00 -> 15.9 mm
- net /SW_RESET: track 0.00 -> 15.1 mm
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- added copper zone on B.Cu, net GND

Commit message: routing
Parts:
- S2: value RESET -> VOL-
- S3: value VOLUME+ -> MUTE
- S4: value VOLUME- -> RESET
- S5: value BASS+ -> BASS-
- S6: value BASS- -> BASS+
- S8: value PROG2 -> VOL+
- moved R11 1.32 mm to (139.7, 138.9), turned to -90 degrees
- moved C12 1.02 mm to (149.4, 106.7)
- moved C11 0.89 mm to (152.5, 106.7)
Connections:
- C2 pad 1: /SW_RESET -> /SW_VOLM
- C3 pad 1: /SW_VOLP -> /SW_MUTE
- C4 pad 1: /SW_VOLM -> /SW_RESET
- C5 pad 1: /SW_BASSP -> /SW_BASSM
- C6 pad 1: /SW_BASSM -> /SW_BASSP
- C8 pad 1: /SW_PROG2 -> /SW_VOLP
- R10 pad 2: /SW_PROG2 -> /SW_VOLP
- R4 pad 2: /SW_RESET -> /SW_VOLM
- R5 pad 2: /SW_VOLP -> /SW_MUTE
- R6 pad 2: /SW_VOLM -> /SW_RESET
- R7 pad 2: /SW_BASSP -> /SW_BASSM
- R8 pad 2: /SW_BASSM -> /SW_BASSP
- U1 pad 13: /SW_RESET -> /IR_OUT
- U1 pad 16: /SW_PROG2 -> /SW_PROG1
- U1 pad 18: /SW_BASSP -> /SW_MUTE
- U1 pad 19: /SW_BASSM -> /SW_RESET
- U1 pad 20: /SW_PROG1 -> /SW_BASSP
- U1 pad 21: /IR_OUT -> /SW_BASSM
- U1 pad 5: /SW_VOLP -> /SW_VOLM
- U1 pad 6: /SW_VOLM -> /SW_VOLP
Routing:
- net GND: track 12.5 -> 85.8 mm, vias 13 -> 34
- net /SW_MUTE: track 0.00 -> 51.0 mm
- net /SW_RESET: track 15.1 -> 59.2 mm
- net /SW_PROG2: track 30.7 -> 0.00 mm
- net /IR_OUT: track 36.9 -> 67.2 mm
- net /SW_BASSP: track 15.9 -> 45.6 mm
- net /SW_STANDBY: track 45.1 -> 74.5 mm
- net /SW_PROG1: track 5.92 -> 34.2 mm
- net /SW_VOLP: track 25.2 -> 51.2 mm
- net Net-(J1-PadS1): track 0.00 -> 25.8 mm
- net /RST: track 60.1 -> 76.3 mm
- net +3V3: track 369.2 -> 358.5 mm, vias 8 -> 10
- net /SW_BASSM: track 27.1 -> 35.6 mm
- net /SW_VOLM: track 42.3 -> 36.8 mm, vias 0 -> 2
- net VBUS: track 57.6 -> 52.8 mm
- removed copper zone on F.Cu, net GND

Commit message: routing
Parts:
- moved C6 2.33 mm to (127.5, 84.5)
- moved R8 2.33 mm to (129.8, 84.5)
- moved R6 2.29 mm to (129.8, 71.1)
- moved R7 2.11 mm to (129.7, 97.6)
- moved R9 2.03 mm to (149.9, 98.0)
- moved C4 1.07 mm to (127.0, 71.1)
- moved C7 1.02 mm to (147.1, 98.1)
- moved C5 0.70 mm to (126.8, 97.7)
Routing:
- net /RST: track 76.3 -> 71.1 mm
- net /SW_PROG1: track 34.2 -> 31.2 mm
- net /SW_BASSP: track 45.6 -> 47.5 mm
- net Net-(R6-Pad1): track 10.7 -> 9.35 mm
- net Net-(R7-Pad1): track 10.6 -> 9.46 mm
- net /SW_RESET: track 59.2 -> 60.1 mm
- net Net-(R9-Pad1): track 10.8 -> 9.92 mm
- net /SW_BASSM: track 35.6 -> 36.2 mm
- net Net-(R8-Pad1): track 10.1 -> 9.61 mm
- net /SW_VOLM: track 36.8 -> 36.4 mm, vias 2 -> 0
Other:
- outline, holes or cut-outs redrawn

Commit message: routing
Parts:
- moved R5 2.55 mm to (149.6, 83.8)
- moved R10 2.03 mm to (169.4, 83.8)
- moved R3 2.03 mm to (169.4, 69.8)
- moved C3 1.30 mm to (146.8, 83.8)
- moved C1 1.02 mm to (166.9, 69.8)
- moved R4 1.02 mm to (169.9, 97.8)
- moved J2 0.72 mm to (173.2, 123.2)
- moved C8 0.51 mm to (166.9, 83.8)
Routing:
- net /RST: track 71.1 -> 75.0 mm
- net /SW_MUTE: track 51.0 -> 48.5 mm
- net +3V3: track 358.4 -> 356.3 mm
- net /SW_STANDBY: track 74.3 -> 72.2 mm
- net /SW_VOLP: track 51.2 -> 49.2 mm
- net Net-(R5-Pad1): track 10.4 -> 8.91 mm
- net /SW_VOLM: track 36.4 -> 35.4 mm
- net Net-(R10-Pad1): track 9.81 -> 8.91 mm
- net Net-(R3-Pad1): track 9.81 -> 8.91 mm
- net /TXD0: track 25.9 -> 25.0 mm
- net /BOOT0: track 42.5 -> 41.7 mm
- net /BOOT1: track 55.4 -> 54.7 mm
- net VBUS: track 52.8 -> 52.0 mm
- net /RXD0: track 27.6 -> 27.1 mm
