File: hardware/ble_ir_remote.kicad_pcb (KiCad board)
At the start: 2 copper layers, 61 x 90.7 mm, 44 parts, among them J1 TYPE-C-31-M-12, J2 Debug connector, Q1 MMBT3904, U1 ESP32-C3-MINI-1-N4, U2 XC6206PxxxMR, U3 SRV05-4

Commit message: cleanup
Routing:
- net GND: track 91.8 -> 99.2 mm, vias 34 -> 27
Changed lines of the file:
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@@
   (segment (start 126.8222 96.9012) (end 126.8222 95.5172) (width 0.2) (layer "F.Cu") (net 17))
   (segment (start 150.902 105.892) (end 150.902 105.055) (width 0.2) (layer "F.Cu") (net 17))
+  (segment (start 151.675 115.881) (end 147.725 115.881) (width 0.2) (layer "F.Cu") (net 17))
   (segment (start 144.8 111.956) (end 144.75 111.906) (width 0.2) (layer "F.Cu") (net 17))
   (segment (start 154.65 111.906) (end 154.65 113.006) (width 0.2) (layer "F.Cu") (net 17))
@@
   (segment (start 144.07 136.7215) (end 142.9845 135.636) (width 0.2) (layer "F.Cu") (net 17))
   (segment (start 154.65 113.006) (end 154.6 113.056) (width 0.2) (layer "F.Cu") (net 17))
-  (segment (start 147.725 115.881) (end 151.675 115.881) (width 0.2) (layer "F.Cu") (net 17))
   (segment (start 152.527 105.905) (end 152.514 105.892) (width 0.2) (layer "F.Cu") (net 17))
   (segment (start 154.6 122.656) (end 153.644 122.656) (width 0.2) (layer "F.Cu") (net 17))
   (segment (start 132.9205 129.606) (end 132.9205 128.3185) (width 0.2) (layer "F.Cu") (net 17))
   (segment (start 151.638 119.868) (end 151.675 119.831) (width 0.2) (layer "F.Cu") (net 17))
+  (segment (start 147.69 121.65) (end 147.69 119.866) (width 0.2) (layer "F.Cu") (net 17))
+  (segment (start 151.675 114.205) (end 151.57 114.1) (width 0.2) (layer "F.Cu") (net 17))
+  (segment (start 149.7 119.831) (end 149.7 115.881) (width 0.2) (layer "F.Cu") (net 17))
   (segment (start 151.675 119.724) (end 151.638 119.761) (width 0.2) (layer "F.Cu") (net 17))
-  (segment (start 152.9 111.956) (end 152.9 113.022) (width 0.2) (layer "F.Cu") (net 17))
   (segment (start 153.644 122.656) (end 153.162 122.174) (width 0.2) (layer "F.Cu") (net 17))
+  (segment (start 152.9 110.54) (end 153.67 109.77) (width 0.2) (layer "F.Cu") (net 17))
   (segment (start 152.842 64.6915) (end 152.842 66.101) (width 0.2) (layer "F.Cu") (net 17))
   (segment (start 156.52 140.1) (end 156.52 138.867) (width 0.2) (layer "F.Cu") (net 17))
@@
   (segment (start 154.6 113.056) (end 154.6 113.856) (width 0.2) (layer "F.Cu") (net 17))
   (segment (start 147.701 114.173) (end 147.701 115.951) (width 0.2) (layer "F.Cu") (net 17))
+  (segment (start 142.63 115.07) (end 143.044 114.656) (width 0.2) (layer "F.Cu") (net 17))
   (segment (start 154.6 117.856) (end 151.675 117.856) (width 0.2) (layer "F.Cu") (net 17))
   (segment (start 132.9205 128.3185) (end 132.969 128.27) (width 0.2) (layer "F.Cu") (net 17))
@@
   (segment (start 150.902 105.892) (end 149.352 105.892) (width 0.2) (layer "F.Cu") (net 17))
   (segment (start 145.1555 129.286) (end 144.807283 129.286) (width 0.2) (layer "F.Cu") (net 17))
-  (segment (start 151.568 119.831) (end 147.725 119.831) (width 0.2) (layer "F.Cu") (net 17))
   (segment (start 144.75 123.806) (end 142.896 123.806) (width 0.2) (layer "F.Cu") (net 17))
-  (segment (start 147.73 119.78) (end 147.725 119.775) (width 0.2) (layer "F.Cu") (net 17))
+  (segment (start 147.725 117.856) (end 151.675 117.856) (width 0.2) (layer "F.Cu") (net 17))
   (segment (start 142.9845 135.636) (end 142.494 135.636) (width 0.2) (layer "F.Cu") (net 17))
   (segment (start 154.65 111.906) (end 152.95 111.906) (width 0.2) (layer "F.Cu") (net 17))
   (segment (start 144.07 129.48) (end 144.07 132.16) (width 0.2) (layer "F.Cu") (net 17))
   (segment (start 152.514 105.892) (end 150.902 105.892) (width 0.2) (layer "F.Cu") (net 17))
-  (segment (start 147.725 119.775) (end 147.725 115.881) (width 0.2) (layer "F.Cu") (net 17))
   (segment (start 144.07 132.16) (end 143.96 132.27) (width 0.2) (layer "F.Cu") (net 17))
   (segment (start 152.95 111.906) (end 152.9 111.956) (width 0.2) (layer "F.Cu") (net 17))
-  (segment (start 142.406 114.656) (end 144.8 114.656) (width 0.2) (layer "F.Cu") (net 17))
-  (segment (start 152.9 113.022) (end 152.908 113.03) (width 0.2) (layer "F.Cu") (net 17))
+  (segment (start 147.725 119.831) (end 151.675 119.831) (width 0.2) (layer "F.Cu") (net 17))
+  (segment (start 147.69 119.866) (end 147.725 119.831) (width 0.2) (layer "F.Cu") (net 17))
+  (segment (start 152.9 111.956) (end 152.9 110.54) (width 0.2) (layer "F.Cu") (net 17))
+  (segment (start 147.725 119.831) (end 147.725 115.881) (width 0.2) (layer "F.Cu") (net 17))
+  (segment (start 143.044 114.656) (end 144.8 114.656) (width 0.2) (layer "F.Cu") (net 17))
   (segment (start 151.227 89.565) (end 143.812 89.565) (width 0.25) (layer "F.Cu") (net 17))
-  (segment (start 142.36 114.61) (end 142.406 114.656) (width 0.2) (layer "F.Cu") (net 17))
   (segment (start 166.878 83.032) (end 166.878 81.788) (width 0.2) (layer "F.Cu") (net 17))
   (segment (start 144.26 129.29) (end 144.07 129.48) (width 0.2) (layer "F.Cu") (net 17))
@@
   (segment (start 144.75 111.906) (end 144.75 110.393) (width 0.2) (layer "F.Cu") (net 17))
   (segment (start 151.638 117.856) (end 151.765 117.729) (width 0.2) (layer "F.Cu") (net 17))
+  (segment (start 151.675 115.881) (end 151.675 114.205) (width 0.2) (layer "F.Cu") (net 17))
   (segment (start 151.257 89.535) (end 151.227 89.565) (width 0.25) (layer "F.Cu") (net 17))
   (segment (start 128.016 129.781) (end 128.016 128.397) (width 0.2) (layer "F.Cu") (net 17))
@@
   (segment (start 139.7 138.049) (end 139.7 136.779) (width 0.2) (layer "F.Cu") (net 17))
   (segment (start 139.192 129.006) (end 139.192 127.635) (width 0.2) (layer "F.Cu") (net 17))
-  (segment (start 149.93 115.881) (end 151.675 115.881) (width 0.2) (layer "F.Cu") (net 17))
   (segment (start 127.508 83.744) (end 126.124 83.744) (width 0.2) (layer "F.Cu") (net 17))
   (segment (start 144.75 110.393) (end 144.78 110.363) (width 0.2) (layer "F.Cu") (net 17))
@@
   (segment (start 150.57 135.434) (end 151.13 134.874) (width 0.2) (layer "F.Cu") (net 17))
   (segment (start 167.132 97.028) (end 167.132 95.758) (width 0.2) (layer "F.Cu") (net 17))
-  (segment (start 147.828 117.856) (end 151.638 117.856) (width 0.2) (layer "F.Cu") (net 17))
   (segment (start 156.52 138.867) (end 156.464 138.811) (width 0.2) (layer "F.Cu") (net 17))
   (segment (start 154.6 117.056) (end 154.6 122.656) (width 0.2) (layer "F.Cu") (net 17))
   (via (at 126.111 83.757) (size 0.8) (drill 0.4) (layers "F.Cu" "B.Cu") (net 17))
-  (via (at 147.828 117.856) (size 0.8) (drill 0.4) (layers "F.Cu" "B.Cu") (net 17))
   (via (at 151.257 89.535) (size 0.8) (drill 0.4) (layers "F.Cu" "B.Cu") (free) (net 17))
-  (via (at 147.701 115.951) (size 0.8) (drill 0.4) (layers "F.Cu" "B.Cu") (net 17))
   (via (at 146.812 81.788) (size 0.8) (drill 0.4) (layers "F.Cu" "B.Cu") (net 17))
   (via (at 166.878 81.788) (size 0.8) (drill 0.4) (layers "F.Cu" "B.Cu") (net 17))
   (via (at 126.8222 95.5172) (size 0.8) (drill 0.4) (layers "F.Cu" "B.Cu") (net 17))
-  (via (at 151.638 119.761) (size 0.8) (drill 0.4) (layers "F.Cu" "B.Cu") (net 17))
   (via (at 144.78 110.363) (size 0.8) (drill 0.4) (layers "F.Cu" "B.Cu") (net 17))
   (via (at 151.13 134.874) (size 0.8) (drill 0.4) (layers "F.Cu" "B.Cu") (net 17))
   (via (at 166.878 67.818) (size 0.8) (drill 0.4) (layers "F.Cu" "B.Cu") (net 17))
-  (via (at 151.675 115.881) (size 0.8) (drill 0.4) (layers "F.Cu" "B.Cu") (net 17))
-  (via (at 149.93 115.881) (size 0.8) (drill 0.4) (layers "F.Cu" "B.Cu") (net 17))
+  (via (at 151.57 114.1) (size 0.8) (drill 0.4) (layers "F.Cu" "B.Cu") (net 17))
   (via (at 128.016 128.397) (size 0.8) (drill 0.4) (layers "F.Cu" "B.Cu") (net 17))
   (via (at 127 69.088) (size 0.8) (drill 0.4) (layers "F.Cu" "B.Cu") (net 17))
-  (via (at 149.733 117.856) (size 0.8) (drill 0.4) (layers "F.Cu" "B.Cu") (net 17))
   (via (at 153.162 122.174) (size 0.8) (drill 0.4) (layers "F.Cu" "B.Cu") (net 17))
   (via (at 139.7 136.779) (size 0.8) (drill 0.4) (layers "F.Cu" "B.Cu") (net 17))
@@
   (via (at 142.89 123.8) (size 0.8) (drill 0.4) (layers "F.Cu" "B.Cu") (free) (net 17))
   (via (at 156.464 138.811) (size 0.8) (drill 0.4) (layers "F.Cu" "B.Cu") (net 17))
-  (via (at 149.733 119.761) (size 0.8) (drill 0.4) (layers "F.Cu" "B.Cu") (net 17))
-  (via (at 152.908 113.03) (size 0.8) (drill 0.4) (layers "F.Cu" "B.Cu") (net 17))
+  (via (at 153.67 109.77) (size 0.8) (drill 0.4) (layers "F.Cu" "B.Cu") (net 17))
   (via (at 139.192 127.635) (size 0.8) (drill 0.4) (layers "F.Cu" "B.Cu") (net 17))
   (via (at 142.494 135.636) (size 0.8) (drill 0.4) (layers "F.Cu" "B.Cu") (net 17))
@@
   (via (at 167.132 95.758) (size 0.8) (drill 0.4) (layers "F.Cu" "B.Cu") (net 17))
   (via (at 151.638 121.666) (size 0.8) (drill 0.4) (layers "F.Cu" "B.Cu") (net 17))
-  (via (at 147.73 119.78) (size 0.8) (drill 0.4) (layers "F.Cu" "B.Cu") (net 17))
+  (via (at 147.69 121.65) (size 0.8) (drill 0.4) (layers "F.Cu" "B.Cu") (net 17))
   (via (at 143.96 132.27) (size 0.8) (drill 0.4) (layers "F.Cu" "B.Cu") (net 17))
   (via (at 147.701 114.173) (size 0.8) (drill 0.4) (layers "F.Cu" "B.Cu") (net 17))
-  (via (at 142.36 114.61) (size 0.8) (drill 0.4) (layers "F.Cu" "B.Cu") (free) (net 17))
-  (via (at 151.765 117.729) (size 0.8) (drill 0.4) (layers "F.Cu" "B.Cu") (net 17))
+  (via (at 142.63 115.07) (size 0.8) (drill 0.4) (layers "F.Cu" "B.Cu") (free) (net 17))
   (segment (start 145.1555 130.9315) (end 145.542 131.318) (width 0.2) (layer "F.Cu") (net 18))
   (segment (start 147.3 123.756) (end 147.3 130.56) (width 0.2) (layer "F.Cu") (net 18))

Commit message: cleanup
Parts:
- added C13: 10u, Capacitor_SMD:C_0603_1608Metric, F.Cu at (152.3, 109.2)
- added C14: 100n, Capacitor_SMD:C_0603_1608Metric, F.Cu at (119.9, 65.3)
- added C15: 100n, Capacitor_SMD:C_0603_1608Metric, F.Cu at (160.0, 78.7)
- moved C12 3.04 mm to (152.3, 106.0), turned to 0 degrees
- moved C11 0.98 mm to (152.3, 107.6), turned to 0 degrees
Routing:
- net GND: track 99.2 -> 103.4 mm, vias 27 -> 28

Commit message: fixes
Parts:
- R9: value 10K -> 1K
- moved D1 2.55 mm to (147.8, 55.9), turned to 180 degrees
Connections:
- D1 pad 2: Net-(D1-Pad2) -> Net-(R2-Pad2)
- Q1 pad 3: Net-(D1-Pad2) -> Net-(D1-Pad1)
- R2 pad 2: Net-(D1-Pad1) -> Net-(R2-Pad2)
Routing:
- net Net-(D1-Pad2): track 10.1 -> 0.00 mm
- net Net-(D1-Pad1): track 2.73 -> 10.1 mm
- net Net-(R2-Pad2): track 0.00 -> 2.73 mm
Other:
- board size 61 x 90.7 mm -> 61 x 90.9 mm
- board text added: "↑"
Changed lines of the file:
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@@
   (net 0 "")
   (net 1 "Net-(D1-Pad1)")
-  (net 2 "Net-(D1-Pad2)")
+  (net 2 "Net-(R2-Pad2)")
   (net 3 "unconnected-(U1-Pad4)")
   (net 4 "/SW_STANDBY")
@@
       (effects (font (size 1 1) (thickness 0.15)))
     )
-    (fp_text value "10K" (at -0.508 -2.794 90) (layer "F.Fab")
+    (fp_text value "1K" (at 0 -2.794 90) (layer "F.Fab")
       (effects (font (size 1 1) (thickness 0.15)))
     )
@@
   )
   (footprint "LED_THT:LED_D3.0mm_IRBlack" (layer "F.Cu")
-    (at 145.283 55.88)
+    (at 147.828 55.88 180)
     (descr "IR-ED, diameter 3.0mm, 2 pins, color: black")
     (tags "IR infrared LED diameter 3.0mm 2 pins black")
@@
     (property "Sheetname" "")
     (attr through_hole)
-    (fp_text reference "D1" (at 4.831 -1.016) (layer "F.SilkS")
-      (effects (font (size 1 1) (thickness 0.15)))
-    )
-    (fp_text value "TSAL6200" (at 1.27 2.96) (layer "F.Fab")
+    (fp_text reference "D1" (at -2.286 -0.762) (layer "F.SilkS")
+      (effects (font (size 1 1) (thickness 0.15)))
+    )
+    (fp_text value "TSAL6200" (at 1.27 -3.302) (layer "F.Fab")
       (effects (font (size 1 1) (thickness 0.15)))
     )
@@
     (fp_arc (start -0.23 -1.16619) (mid 3.17 0.000452) (end -0.230555 1.165476) (layer "F.Fab") (width 0.1))
     (fp_circle (center 1.27 0) (end 2.77 0) (layer "F.Fab") (width 0.1) (fill none))
-    (pad "1" thru_hole rect (at 0 0) (size 1.8 1.8) (drill 0.9) (layers *.Cu *.Mask)
+    (pad "1" thru_hole rect (at 0 0 180) (size 1.8 1.8) (drill 0.9) (layers *.Cu *.Mask)
       (net 1 "Net-(D1-Pad1)") (pinfunction "K") (pintype "passive"))
-    (pad "2" thru_hole circle (at 2.54 0) (size 1.8 1.8) (drill 0.9) (layers *.Cu *.Mask)
-      (net 2 "Net-(D1-Pad2)") (pinfunction "A") (pintype "passive"))
+    (pad "2" thru_hole circle (at 2.54 0 180) (size 1.8 1.8) (drill 0.9) (layers *.Cu *.Mask)
+      (net 2 "Net-(R2-Pad2)") (pinfunction "A") (pintype "passive"))
     (model "${KICAD6_3DMODEL_DIR}/LED_THT.3dshapes/LED_D3.0mm_IRBlack.wrl"
       (offset (xyz 0 0 0))
@@
       (net 17 "GND") (pinfunction "E") (pintype "passive"))
     (pad "3" smd roundrect (at 0.9375 0 90) (size 1.475 0.6) (layers "F.Cu" "F.Paste" "F.Mask") (roundrect_rratio 0.25)
-      (net 2 "Net-(D1-Pad2)") (pinfunction "C") (pintype "passive"))
+      (net 1 "Net-(D1-Pad1)") (pinfunction "C") (pintype "passive"))
     (model "${KICAD6_3DMODEL_DIR}/Package_TO_SOT_SMD.3dshapes/SOT-23.wrl"
       (offset (xyz 0 0 0))
@@
       (net 32 "+3V3") (pintype "passive"))
     (pad "2" smd roundrect (at 0.825 0) (size 0.8 0.95) (layers "F.Cu" "F.Paste" "F.Mask") (roundrect_rratio 0.25)
-      (net 1 "Net-(D1-Pad1)") (pintype "passive"))
+      (net 2 "Net-(R2-Pad2)") (pintype "passive"))
     (model "${KICAD6_3DMODEL_DIR}/Resistor_SMD.3dshapes/R_0603_1608Metric.wrl"
       (offset (xyz 0 0 0))
@@
     )
   )
-  (gr_arc (start 177.038 142.748) (mid 176.666026 143.646026) (end 175.768 144.018) (layer "Edge.Cuts") (width 0.1))
-  (gr_arc (start 118.11 144.018) (mid 116.673159 143.422841) (end 116.078 141.986) (layer "Edge.Cuts") (width 0.1))
-  (gr_line (start 116.078 141.986) (end 116.078 55.118) (layer "Edge.Cuts") (width 0.1))
+  (gr_arc (start 177.038 143.002) (mid 176.666026 143.900026) (end 175.768 144.272) (layer "Edge.Cuts") (width 0.1))
+  (gr_arc (start 118.11 144.272) (mid 116.673159 143.676841) (end 116.078 142.24) (layer "Edge.Cuts") (width 0.1))
+  (gr_line (start 116.078 142.24) (end 116.078 55.118) (layer "Edge.Cuts") (width 0.1))
   (gr_arc (start 116.078 55.118) (mid 116.598764 53.860764) (end 117.856 53.34) (layer "Edge.Cuts") (width 0.1))
   (gr_arc (start 175.26 53.34) (mid 176.424949 53.774803) (end 177.02013 54.866553) (layer "Edge.Cuts") (width 0.1))
-  (gr_line (start 177.02013 54.866553) (end 177.038 142.748) (layer "Edge.Cuts") (width 0.1))
+  (gr_line (start 177.02013 54.866553) (end 177.038 143.002) (layer "Edge.Cuts") (width 0.1))
   (gr_line (start 117.856 53.34) (end 175.26 53.34) (layer "Edge.Cuts") (width 0.1))
-  (gr_line (start 175.768 144.018) (end 118.11 144.018) (layer "Edge.Cuts") (width 0.1))
+  (gr_line (start 175.768 144.272) (end 118.11 144.272) (layer "Edge.Cuts") (width 0.1))
   (gr_rect (start 161.036 124.968) (end 155.194 110.744) (layer "Edge.Cuts") (width 0.1) (fill none))
-  (segment (start 142.557 55.88) (end 145.283 55.88) (width 0.2) (layer "F.Cu") (net 1))
-  (segment (start 151.892 57.404) (end 151.892 62.8165) (width 0.2) (layer "F.Cu") (net 2))
-  (segment (start 147.823 55.88) (end 150.368 55.88) (width 0.2) (layer "F.Cu") (net 2))
-  (segment (start 150.368 55.88) (end 151.892 57.404) (width 0.2) (layer "F.Cu") (net 2))
+  (gr_text "↑" (at 149.606 54.356) (layer "F.SilkS")
+    (effects (font (size 1 1) (thickness 0.15)))
+  )
+  (dimension (type aligned) (layer "F.SilkS")
+    (pts (xy 116.09 49.8) (xy 177.08 49.82))
+    (height -4.251058)
+    (gr_text "60.9900 mm" (at 146.586771 44.408942 359.9812114) (layer "F.SilkS")
+      (effects (font (size 1 1) (thickness 0.15)))
+    )
+    (format (units 3) (units_format 1) (precision 4))
+    (style (thickness 0.15) (arrow_length 1.27) (text_position_mode 0) (extension_height 0.58642) (extension_offset 0.5) keep_text_aligned)
+  )
+  (dimension (type aligned) (layer "F.SilkS")
+    (pts (xy 182.06 144.22) (xy 182.06 53.31))
+    (height 8.23)
+    (gr_text "90.9100 mm" (at 189.14 98.765 90) (layer "F.SilkS")
+      (effects (font (size 1 1) (thickness 0.15)))
+    )
+    (format (units 3) (units_format 1) (precision 4))
+    (style (thickness 0.15) (arrow_length 1.27) (text_position_mode 0) (extension_height 0.58642) (extension_offset 0.5) keep_text_aligned)
+  )
+  (segment (start 151.892 57.404) (end 151.892 62.8165) (width 0.2) (layer "F.Cu") (net 1))
+  (segment (start 147.823 55.88) (end 150.368 55.88) (width 0.2) (layer "F.Cu") (net 1))
+  (segment (start 150.368 55.88) (end 151.892 57.404) (width 0.2) (layer "F.Cu") (net 1))
+  (segment (start 142.557 55.88) (end 145.283 55.88) (width 0.2) (layer "F.Cu") (net 2))
   (segment (start 158.785 70.675) (end 157.05 72.41) (width 0.2) (layer "F.Cu") (net 4))
   (segment (start 142.289 101.551) (end 156.669 101.551) (width 0.2) (layer "F.Cu") (net 4))
