File: hardware/ble_ir_remote.kicad_sch (KiCad schematic)
At the start: 42 parts, among them J1 TYPE-C-31-M-12, J2 Debug connector, Q1 MMBT3904, U2 XC6206PxxxMR, U3 SRV05-4

Commit message: routing
Parts:
- C11, C9: value (none) -> 10u
- U1: value (none) -> ESP32-C3-MINI-1-N4; footprint (none) -> XCVR_ESP32-C3-MINI-1-N4
Connections:
- net BOOT0: now also J2.5 (Pin_5); no longer J2.6 (Pin_6)
- net BOOT1: now also J2.6 (Pin_6); no longer J2.7 (Pin_7)
- net GND: now also J2.1 (Pin_1); no longer J2.8 (Pin_8)
- net RST: now also J2.7 (Pin_7); no longer J2.3 (Pin_3)
- net TXD0: now also J2.3 (Pin_3); no longer J2.5 (Pin_5)
- net VBUS: now also J2.8 (Pin_8); no longer J2.1 (Pin_1)
Changed lines of the file:
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@@
-    (stroke (width 0) (type default) (color 0 0 0 0))
-  )
-  (wire (pts (xy 50.8 155.575) (xy 57.785 155.575))
     (stroke (width 0) (type default) (color 0 0 0 0))
   )
@@
     (stroke (width 0) (type default) (color 0 0 0 0))
   )
-  (wire (pts (xy 50.8 158.115) (xy 63.5 158.115))
-    (stroke (width 0) (type default) (color 0 0 0 0))
-  )
   (wire (pts (xy 257.175 69.85) (xy 260.985 69.85))
     (stroke (width 0) (type default) (color 0 0 0 0))
@@
     (stroke (width 0) (type default) (color 0 0 0 0))
   )
-  (wire (pts (xy 63.5 158.115) (xy 63.5 151.765))
-    (stroke (width 0) (type default) (color 0 0 0 0))
-  )
   (wire (pts (xy 65.405 29.21) (xy 65.405 24.13))
     (stroke (width 0) (type default) (color 0 0 0 0))
@@
     (stroke (width 0) (type default) (color 0 0 0 0))
   )
-  (wire (pts (xy 57.785 155.575) (xy 57.785 151.765))
-    (stroke (width 0) (type default) (color 0 0 0 0))
-  )
   (wire (pts (xy 172.085 64.77) (xy 172.085 62.865))
     (stroke (width 0) (type default) (color 0 0 0 0))
@@
     (effects (font (size 1.27 1.27)) (justify left bottom))
   )
-  (label "BOOT0" (at 50.8 168.275 0)
+  (label "BOOT0" (at 50.8 165.735 0)
     (effects (font (size 1.27 1.27)) (justify left bottom))
   )
@@
     (effects (font (size 1.27 1.27)) (justify right bottom))
   )
-  (label "TXD0" (at 50.8 165.735 0)
+  (label "TXD0" (at 50.8 160.655 0)
     (effects (font (size 1.27 1.27)) (justify left bottom))
   )
@@
     (effects (font (size 1.27 1.27)) (justify left bottom))
   )
-  (label "RST" (at 50.8 160.655 0)
+  (label "RST" (at 50.8 170.815 0)
     (effects (font (size 1.27 1.27)) (justify left bottom))
   )
@@
     (effects (font (size 1.27 1.27)) (justify left bottom))
   )
-  (label "BOOT1" (at 50.8 170.815 0)
+  (label "BOOT1" (at 50.8 168.275 0)
     (effects (font (size 1.27 1.27)) (justify left bottom))
   )
@@
       (effects (font (size 1.27 1.27)) (justify right))
     )
-    (property "Value" "" (id 1) (at 130.81 109.8485 0)
+    (property "Value" "10u" (id 1) (at 130.81 109.8485 0)
       (effects (font (size 1.27 1.27)) (justify right))
     )
@@
     (pin "1")
   )
-  (symbol (lib_id "power:VBUS") (at 57.785 151.765 0) (unit 1)
+  (symbol (lib_id "power:VBUS") (at 50.8 173.355 270) (unit 1)
     (in_bom yes) (on_board yes)
-    (property "Reference" "#PWR0113" (id 0) (at 57.785 155.575 0)
-      (effects (font (size 1.27 1.27)) hide)
-    )
-    (property "Value" "VBUS" (id 1) (at 55.245 147.32 0)
+    (property "Reference" "#PWR0113" (id 0) (at 46.99 173.355 0)
+      (effects (font (size 1.27 1.27)) hide)
+    )
+    (property "Value" "VBUS" (id 1) (at 55.245 170.815 0)
       (effects (font (size 1.27 1.27)) (justify left))
     )
-    (property "Footprint" "" (id 2) (at 57.785 151.765 0)
-      (effects (font (size 1.27 1.27)) hide)
-    )
-    (property "Datasheet" "" (id 3) (at 57.785 151.765 0)
+    (property "Footprint" "" (id 2) (at 50.8 173.355 0)
+      (effects (font (size 1.27 1.27)) hide)
+    )
+    (property "Datasheet" "" (id 3) (at 50.8 173.355 0)
       (effects (font (size 1.27 1.27)) hide)
     )
@@
     (pin "2")
   )
-  (symbol (lib_id "power:+3V3") (at 63.5 151.765 0) (unit 1)
+  (symbol (lib_id "power:+3V3") (at 50.8 158.115 270) (unit 1)
     (in_bom yes) (on_board yes)
-    (property "Reference" "#PWR0106" (id 0) (at 63.5 155.575 0)
-      (effects (font (size 1.27 1.27)) hide)
-    )
-    (property "Value" "+3V3" (id 1) (at 63.5 147.32 0))
-    (property "Footprint" "" (id 2) (at 63.5 151.765 0)
-      (effects (font (size 1.27 1.27)) hide)
-    )
-    (property "Datasheet" "" (id 3) (at 63.5 151.765 0)
+    (property "Reference" "#PWR0106" (id 0) (at 46.99 158.115 0)
+      (effects (font (size 1.27 1.27)) hide)
+    )
+    (property "Value" "+3V3" (id 1) (at 55.245 158.115 0))
+    (property "Footprint" "" (id 2) (at 50.8 158.115 0)
+      (effects (font (size 1.27 1.27)) hide)
+    )
+    (property "Datasheet" "" (id 3) (at 50.8 158.115 0)
       (effects (font (size 1.27 1.27)) hide)
     )
@@
     (pin "1")
   )
-  (symbol (lib_id "power:GND") (at 50.8 173.355 0) (unit 1)
-    (in_bom yes) (on_board yes) (fields_autoplaced)
-    (property "Reference" "#PWR0105" (id 0) (at 50.8 179.705 0)
-      (effects (font (size 1.27 1.27)) hide)
-    )
-    (property "Value" "GND" (id 1) (at 52.705 174.6249 0)
-      (effects (font (size 1.27 1.27)) (justify left))
-    )
-    (property "Footprint" "" (id 2) (at 50.8 173.355 0)
-      (effects (font (size 1.27 1.27)) hide)
-    )
-    (property "Datasheet" "" (id 3) (at 50.8 173.355 0)
+  (symbol (lib_id "power:GND") (at 50.8 155.575 90) (unit 1)
+    (in_bom yes) (on_board yes)
+    (property "Reference" "#PWR0105" (id 0) (at 57.15 155.575 0)
+      (effects (font (size 1.27 1.27)) hide)
+    )
+    (property "Value" "GND" (id 1) (at 50.165 153.035 90)
+      (effects (font (size 1.27 1.27)) (justify right))
+    )
+    (property "Footprint" "" (id 2) (at 50.8 155.575 0)
+      (effects (font (size 1.27 1.27)) hide)
+    )
+    (property "Datasheet" "" (id 3) (at 50.8 155.575 0)
       (effects (font (size 1.27 1.27)) hide)
     )
@@
     (in_bom yes) (on_board yes) (fields_autoplaced)
     (property "Reference" "U1" (id 0) (at 134.62 50.165 0))
-    (property "Value" "" (id 1) (at 134.62 52.705 0))
-    (property "Footprint" "" (id 2) (at 134.62 73.025 0)
+    (property "Value" "ESP32-C3-MINI-1-N4" (id 1) (at 134.62 52.705 0))
+    (property "Footprint" "XCVR_ESP32-C3-MINI-1-N4" (id 2) (at 134.62 73.025 0)
       (effects (font (size 1.27 1.27)) (justify left bottom) hide)
     )
@@
       (effects (font (size 1.27 1.27)) (justify right))
     )
-    (property "Value" "" (id 1) (at 34.29 33.0135 0)
+    (property "Value" "10u" (id 1) (at 34.29 33.0135 0)
       (effects (font (size 1.27 1.27)) (justify right))
     )

Commit message: routing
Parts:
- S2: value RESET -> (none); footprint SW_TS-1187A-B-A-B -> (none)
- S3: value VOLUME+ -> (none); footprint SW_TS-1187A-B-A-B -> (none)
- S4: value VOLUME- -> (none); footprint SW_TS-1187A-B-A-B -> (none)
- S5: value BASS+ -> (none); footprint SW_TS-1187A-B-A-B -> (none)
- S6: value BASS- -> (none); footprint SW_TS-1187A-B-A-B -> (none)
- S8: value PROG2 -> (none)
Connections:
- net IR_OUT: now also U1.13 (IO1); no longer U1.21 (IO7)
- net SW_BASSM: now also C5.1, R7.2, U1.21 (IO7); no longer C6.1, R8.2, U1.19 (IO5)
- net SW_BASSP: now also C6.1, R8.2, U1.20 (IO6); no longer C5.1, R7.2, U1.18 (IO4)
- net SW_PROG1: now also U1.16 (IO10); no longer U1.20 (IO6)
- net SW_RESET: now also C4.1, R6.2, U1.19 (IO5); no longer C2.1, R4.2, U1.13 (IO1)
- net SW_VOLM: now also C2.1, R4.2, U1.5 (IO2); no longer C4.1, R6.2, U1.6 (IO3)
- net SW_VOLP: now also C8.1, R10.2, U1.6 (IO3); no longer C3.1, R5.2, U1.5 (IO2)
- removed net SW_PROG2: C8.1, R10.2, U1.16 (IO10)
- new net SW_MUTE: C3.1, R5.2, U1.18 (IO4)
Changed lines of the file:
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@@
     (effects (font (size 1.27 1.27)) (justify left bottom))
   )
-  (label "IR_OUT" (at 152.4 65.405 0)
-    (effects (font (size 1.27 1.27)) (justify left bottom))
+  (label "IR_OUT" (at 116.84 67.945 180)
+    (effects (font (size 1.27 1.27)) (justify right bottom))
   )
   (label "BOOT0" (at 50.8 165.735 0)
     (effects (font (size 1.27 1.27)) (justify left bottom))
   )
-  (label "SW_PROG1" (at 116.84 80.645 180)
-    (effects (font (size 1.27 1.27)) (justify right bottom))
+  (label "SW_PROG1" (at 152.4 73.025 0)
+    (effects (font (size 1.27 1.27)) (justify left bottom))
   )
   (label "RXD0" (at 116.84 85.725 180)
     (effects (font (size 1.27 1.27)) (justify right bottom))
   )
-  (label "SW_PROG2" (at 269.24 120.65 90)
-    (effects (font (size 1.27 1.27)) (justify left bottom))
-  )
-  (label "SW_VOLP" (at 116.84 70.485 180)
+  (label "SW_MUTE" (at 268.605 58.42 90)
+    (effects (font (size 1.27 1.27)) (justify left bottom))
+  )
+  (label "SW_MUTE" (at 116.84 75.565 180)
     (effects (font (size 1.27 1.27)) (justify right bottom))
   )
-  (label "SW_BASSM" (at 269.24 93.98 90)
+  (label "SW_VOLP" (at 116.84 73.025 180)
+    (effects (font (size 1.27 1.27)) (justify right bottom))
+  )
+  (label "SW_BASSM" (at 269.24 81.28 90)
     (effects (font (size 1.27 1.27)) (justify left bottom))
   )
@@
     (effects (font (size 1.27 1.27)) (justify left bottom))
   )
-  (label "SW_VOLM" (at 269.24 69.85 90)
+  (label "SW_VOLM" (at 268.605 45.72 90)
     (effects (font (size 1.27 1.27)) (justify left bottom))
   )
@@
     (effects (font (size 1.27 1.27)) (justify left bottom))
   )
-  (label "SW_BASSP" (at 116.84 75.565 180)
+  (label "SW_BASSP" (at 116.84 80.645 180)
     (effects (font (size 1.27 1.27)) (justify right bottom))
   )
-  (label "SW_RESET" (at 269.24 45.72 90)
+  (label "SW_RESET" (at 268.605 69.85 90)
     (effects (font (size 1.27 1.27)) (justify left bottom))
   )
@@
     (effects (font (size 1.27 1.27)) (justify right bottom))
   )
-  (label "SW_VOLM" (at 116.84 73.025 180)
+  (label "SW_VOLM" (at 116.84 70.485 180)
     (effects (font (size 1.27 1.27)) (justify right bottom))
   )
@@
     (effects (font (size 1.27 1.27)) (justify right bottom))
   )
-  (label "SW_RESET" (at 116.84 67.945 180)
+  (label "SW_RESET" (at 116.84 78.105 180)
     (effects (font (size 1.27 1.27)) (justify right bottom))
   )
@@
     (effects (font (size 1.27 1.27)) (justify right bottom))
   )
-  (label "SW_BASSM" (at 116.84 78.105 180)
-    (effects (font (size 1.27 1.27)) (justify right bottom))
-  )
-  (label "SW_VOLP" (at 269.24 58.42 90)
-    (effects (font (size 1.27 1.27)) (justify left bottom))
-  )
-  (label "SW_BASSP" (at 269.24 81.28 90)
+  (label "SW_BASSM" (at 152.4 65.405 0)
+    (effects (font (size 1.27 1.27)) (justify left bottom))
+  )
+  (label "SW_VOLP" (at 269.24 120.65 90)
+    (effects (font (size 1.27 1.27)) (justify left bottom))
+  )
+  (label "SW_BASSP" (at 269.24 93.98 90)
     (effects (font (size 1.27 1.27)) (justify left bottom))
   )
@@
   (label "USB_D+" (at 30.48 66.04 180)
     (effects (font (size 1.27 1.27)) (justify right bottom))
-  )
-  (label "SW_PROG2" (at 152.4 73.025 0)
-    (effects (font (size 1.27 1.27)) (justify left bottom))
   )
   (label "BOOT1" (at 50.8 168.275 0)
@@
     (in_bom yes) (on_board yes)
     (property "Reference" "S2" (id 0) (at 249.555 38.1 0))
-    (property "Value" "RESET" (id 1) (at 249.555 40.64 0))
-    (property "Footprint" "SW_TS-1187A-B-A-B" (id 2) (at 249.555 45.72 0)
+    (property "Value" "" (id 1) (at 249.555 40.64 0))
+    (property "Footprint" "" (id 2) (at 249.555 45.72 0)
       (effects (font (size 1.27 1.27)) (justify left bottom) hide)
     )
@@
     (in_bom yes) (on_board yes)
     (property "Reference" "S6" (id 0) (at 249.555 86.36 0))
-    (property "Value" "BASS-" (id 1) (at 249.555 88.9 0))
-    (property "Footprint" "SW_TS-1187A-B-A-B" (id 2) (at 249.555 93.98 0)
+    (property "Value" "" (id 1) (at 249.555 88.9 0))
+    (property "Footprint" "" (id 2) (at 249.555 93.98 0)
       (effects (font (size 1.27 1.27)) (justify left bottom) hide)
     )
@@
     (in_bom yes) (on_board yes)
     (property "Reference" "S8" (id 0) (at 249.555 113.03 0))
-    (property "Value" "PROG2" (id 1) (at 249.555 115.57 0))
+    (property "Value" "" (id 1) (at 249.555 115.57 0))
     (property "Footprint" "SW_TS-1187A-B-A-B" (id 2) (at 249.555 120.65 0)
       (effects (font (size 1.27 1.27)) (justify left bottom) hide)
@@
     (in_bom yes) (on_board yes)
     (property "Reference" "S4" (id 0) (at 249.555 62.23 0))
-    (property "Value" "VOLUME-" (id 1) (at 249.555 64.77 0))
-    (property "Footprint" "SW_TS-1187A-B-A-B" (id 2) (at 249.555 69.85 0)
+    (property "Value" "" (id 1) (at 249.555 64.77 0))
+    (property "Footprint" "" (id 2) (at 249.555 69.85 0)
       (effects (font (size 1.27 1.27)) (justify left bottom) hide)
     )
@@
     (in_bom yes) (on_board yes)
     (property "Reference" "S5" (id 0) (at 249.555 73.66 0))
-    (property "Value" "BASS+" (id 1) (at 249.555 76.2 0))
-    (property "Footprint" "SW_TS-1187A-B-A-B" (id 2) (at 249.555 81.28 0)
+    (property "Value" "" (id 1) (at 249.555 76.2 0))
+    (property "Footprint" "" (id 2) (at 249.555 81.28 0)
       (effects (font (size 1.27 1.27)) (justify left bottom) hide)
     )
@@
     (in_bom yes) (on_board yes)
     (property "Reference" "S3" (id 0) (at 249.555 50.8 0))
-    (property "Value" "VOLUME+" (id 1) (at 249.555 53.34 0))
-    (property "Footprint" "SW_TS-1187A-B-A-B" (id 2) (at 249.555 58.42 0)
+    (property "Value" "" (id 1) (at 249.555 53.34 0))
+    (property "Footprint" "" (id 2) (at 249.555 58.42 0)
       (effects (font (size 1.27 1.27)) (justify left bottom) hide)
     )
@@
     )
     (path "/070c67c3-5f08-4d00-882d-fd6b5081f42c"
-      (reference "S2") (unit 1) (value "RESET") (footprint "SW_TS-1187A-B-A-B")
+      (reference "S2") (unit 1) (value "VOL-") (footprint "SW_TS-1187A-B-A-B")
     )
     (path "/fdcb820d-b9bc-4b60-b223-6ddc09c6929d"
-      (reference "S3") (unit 1) (value "VOLUME+") (footprint "SW_TS-1187A-B-A-B")
+      (reference "S3") (unit 1) (value "MUTE") (footprint "SW_TS-1187A-B-A-B")
     )
     (path "/c67ac3e4-b92d-4731-a29c-3aa570731610"
-      (reference "S4") (unit 1) (value "VOLUME-") (footprint "SW_TS-1187A-B-A-B")
+      (reference "S4") (unit 1) (value "RESET") (footprint "SW_TS-1187A-B-A-B")
     )
     (path "/f95a5364-1b21-4dfa-a4b5-d841e1a4f69a"
-      (reference "S5") (unit 1) (value "BASS+") (footprint "SW_TS-1187A-B-A-B")
+      (reference "S5") (unit 1) (value "BASS-") (footprint "SW_TS-1187A-B-A-B")
     )
     (path "/8b219eba-2b62-4300-94e2-77b8510c1ff2"
-      (reference "S6") (unit 1) (value "BASS-") (footprint "SW_TS-1187A-B-A-B")
+      (reference "S6") (unit 1) (value "BASS+") (footprint "SW_TS-1187A-B-A-B")
     )
     (path "/5c9b48ae-578a-48ac-8587-bbf011bcefac"
@@
     )
     (path "/c486cd04-ee3c-4ece-988c-6a297d5b401c"
-      (reference "S8") (unit 1) (value "PROG2") (footprint "SW_TS-1187A-B-A-B")
+      (reference "S8") (unit 1) (value "VOL+") (footprint "SW_TS-1187A-B-A-B")
     )
     (path "/ab28c48c-701b-4892-a2b9-8b62bf64ab01"

Commit message: fine tuning
Parts:
- S2: value (none) -> VOL-; footprint (none) -> SW_TS-1187A-B-A-B
- S3: value (none) -> MUTE; footprint (none) -> SW_TS-1187A-B-A-B
- S4: value (none) -> RESET; footprint (none) -> SW_TS-1187A-B-A-B
- S5: value (none) -> BASS-; footprint (none) -> SW_TS-1187A-B-A-B
- S6: value (none) -> BASS+; footprint (none) -> SW_TS-1187A-B-A-B
- S8: value (none) -> VOL+
Changed lines of the file:
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@@
+    (stroke (width 0) (type default) (color 0 0 0 0))
+  )
+  (wire (pts (xy 58.42 158.115) (xy 58.42 156.21))
+    (stroke (width 0) (type default) (color 0 0 0 0))
+  )
+  (wire (pts (xy 50.8 173.355) (xy 60.325 173.355))
     (stroke (width 0) (type default) (color 0 0 0 0))
   )
@@
     (stroke (width 0) (type default) (color 0 0 0 0))
   )
+  (wire (pts (xy 60.325 173.355) (xy 60.325 170.815))
+    (stroke (width 0) (type default) (color 0 0 0 0))
+  )
   (wire (pts (xy 19.685 68.58) (xy 19.685 63.5))
     (stroke (width 0) (type default) (color 0 0 0 0))
@@
   )
   (wire (pts (xy 257.175 106.68) (xy 260.985 106.68))
+    (stroke (width 0) (type default) (color 0 0 0 0))
+  )
+  (wire (pts (xy 50.8 158.115) (xy 58.42 158.115))
     (stroke (width 0) (type default) (color 0 0 0 0))
   )
@@
     (in_bom yes) (on_board yes)
     (property "Reference" "S2" (id 0) (at 249.555 38.1 0))
-    (property "Value" "" (id 1) (at 249.555 40.64 0))
-    (property "Footprint" "" (id 2) (at 249.555 45.72 0)
+    (property "Value" "VOL-" (id 1) (at 249.555 40.64 0))
+    (property "Footprint" "SW_TS-1187A-B-A-B" (id 2) (at 249.555 45.72 0)
       (effects (font (size 1.27 1.27)) (justify left bottom) hide)
     )
@@
     (pin "1")
   )
-  (symbol (lib_id "power:VBUS") (at 50.8 173.355 270) (unit 1)
-    (in_bom yes) (on_board yes)
-    (property "Reference" "#PWR0113" (id 0) (at 46.99 173.355 0)
-      (effects (font (size 1.27 1.27)) hide)
-    )
-    (property "Value" "VBUS" (id 1) (at 55.245 170.815 0)
+  (symbol (lib_id "power:VBUS") (at 60.325 170.815 0) (unit 1)
+    (in_bom yes) (on_board yes)
+    (property "Reference" "#PWR0113" (id 0) (at 60.325 174.625 0)
+      (effects (font (size 1.27 1.27)) hide)
+    )
+    (property "Value" "VBUS" (id 1) (at 57.785 166.37 0)
       (effects (font (size 1.27 1.27)) (justify left))
     )
-    (property "Footprint" "" (id 2) (at 50.8 173.355 0)
-      (effects (font (size 1.27 1.27)) hide)
-    )
-    (property "Datasheet" "" (id 3) (at 50.8 173.355 0)
+    (property "Footprint" "" (id 2) (at 60.325 170.815 0)
+      (effects (font (size 1.27 1.27)) hide)
+    )
+    (property "Datasheet" "" (id 3) (at 60.325 170.815 0)
       (effects (font (size 1.27 1.27)) hide)
     )
@@
     (pin "2")
   )
-  (symbol (lib_id "power:+3V3") (at 50.8 158.115 270) (unit 1)
-    (in_bom yes) (on_board yes)
-    (property "Reference" "#PWR0106" (id 0) (at 46.99 158.115 0)
-      (effects (font (size 1.27 1.27)) hide)
-    )
-    (property "Value" "+3V3" (id 1) (at 55.245 158.115 0))
-    (property "Footprint" "" (id 2) (at 50.8 158.115 0)
-      (effects (font (size 1.27 1.27)) hide)
-    )
-    (property "Datasheet" "" (id 3) (at 50.8 158.115 0)
+  (symbol (lib_id "power:+3V3") (at 58.42 156.21 0) (unit 1)
+    (in_bom yes) (on_board yes)
+    (property "Reference" "#PWR0106" (id 0) (at 58.42 160.02 0)
+      (effects (font (size 1.27 1.27)) hide)
+    )
+    (property "Value" "+3V3" (id 1) (at 58.42 151.765 0))
+    (property "Footprint" "" (id 2) (at 58.42 156.21 0)
+      (effects (font (size 1.27 1.27)) hide)
+    )
+    (property "Datasheet" "" (id 3) (at 58.42 156.21 0)
       (effects (font (size 1.27 1.27)) hide)
     )
@@
     (in_bom yes) (on_board yes)
     (property "Reference" "S6" (id 0) (at 249.555 86.36 0))
-    (property "Value" "" (id 1) (at 249.555 88.9 0))
-    (property "Footprint" "" (id 2) (at 249.555 93.98 0)
+    (property "Value" "BASS+" (id 1) (at 249.555 88.9 0))
+    (property "Footprint" "SW_TS-1187A-B-A-B" (id 2) (at 249.555 93.98 0)
       (effects (font (size 1.27 1.27)) (justify left bottom) hide)
     )
@@
     (in_bom yes) (on_board yes)
     (property "Reference" "S8" (id 0) (at 249.555 113.03 0))
-    (property "Value" "" (id 1) (at 249.555 115.57 0))
+    (property "Value" "VOL+" (id 1) (at 249.555 115.57 0))
     (property "Footprint" "SW_TS-1187A-B-A-B" (id 2) (at 249.555 120.65 0)
       (effects (font (size 1.27 1.27)) (justify left bottom) hide)
@@
     (in_bom yes) (on_board yes)
     (property "Reference" "S4" (id 0) (at 249.555 62.23 0))
-    (property "Value" "" (id 1) (at 249.555 64.77 0))
-    (property "Footprint" "" (id 2) (at 249.555 69.85 0)
+    (property "Value" "RESET" (id 1) (at 249.555 64.77 0))
+    (property "Footprint" "SW_TS-1187A-B-A-B" (id 2) (at 249.555 69.85 0)
       (effects (font (size 1.27 1.27)) (justify left bottom) hide)
     )
@@
   )
   (symbol (lib_id "Connector:Conn_01x08_Male") (at 45.72 163.195 0) (unit 1)
-    (in_bom yes) (on_board yes) (fields_autoplaced)
-    (property "Reference" "J2" (id 0) (at 46.355 149.86 0))
-    (property "Value" "Debug connector" (id 1) (at 46.355 152.4 0))
+    (in_bom yes) (on_board yes)
+    (property "Reference" "J2" (id 0) (at 45.72 146.685 0))
+    (property "Value" "Debug connector" (id 1) (at 45.72 149.225 0))
     (property "Footprint" "Connector_PinHeader_2.54mm:PinHeader_1x08_P2.54mm_Vertical" (id 2) (at 45.72 163.195 0)
       (effects (font (size 1.27 1.27)) hide)
@@
     (in_bom yes) (on_board yes)
     (property "Reference" "S5" (id 0) (at 249.555 73.66 0))
-    (property "Value" "" (id 1) (at 249.555 76.2 0))
-    (property "Footprint" "" (id 2) (at 249.555 81.28 0)
+    (property "Value" "BASS-" (id 1) (at 249.555 76.2 0))
+    (property "Footprint" "SW_TS-1187A-B-A-B" (id 2) (at 249.555 81.28 0)
       (effects (font (size 1.27 1.27)) (justify left bottom) hide)
     )
@@
     (in_bom yes) (on_board yes)
     (property "Reference" "S3" (id 0) (at 249.555 50.8 0))
-    (property "Value" "" (id 1) (at 249.555 53.34 0))
-    (property "Footprint" "" (id 2) (at 249.555 58.42 0)
-      (effects (font (size 1.27 1.27)) (justify left bottom) hide)
-    )
+    (property "Value" "MUTE" (id 1) (at 249.555 53.34 0))
+    (property "Footprint" "SW_TS-1187A-B-A-B" (id 2) (at 249.555 58.42 0)
+      (effects (font (size 1.27 1.27)) (justify left bottom) hide)
+    )
