File: hardware/ble_ir_remote.kicad_sch (KiCad schematic)
At the start: 42 parts, among them J1 TYPE-C-31-M-12, J2 Debug connector, Q1 MMBT3904, U1 ESP32-C3-MINI-1-N4, U2 XC6206PxxxMR, U3 SRV05-4

Commit message: fine tuning
Parts:
- added R15, R16: 10K, Resistor_SMD:R_0603_1608Metric, symbol Device:R_Small
Connections:
- net +3V3: now also C7.2, R15.1, R16.1; no longer S7.A, S7.B
- net GND: now also S7.A, S7.B; no longer C7.2
- net RST: now also R16.2
- net SW_PROG1: now also U1.5 (IO2), R15.2; no longer U1.16 (IO10)
- net SW_VOLM: now also U1.16 (IO10); no longer U1.5 (IO2)
Other:
- moved on the sheet: D2, R13, R14
