File: hardware/ble_ir_remote.kicad_sch (KiCad schematic)
At the start: 44 parts, among them J1 TYPE-C-31-M-12, J2 Debug connector, Q1 MMBT3904, U1 ESP32-C3-MINI-1-N4, U2 XC6206PxxxMR, U3 SRV05-4

Commit message: cleanup
Other:
- moved on the sheet: C11, C12, D2, R13, R14, R15, R16, U1

Commit message: cleanup
Parts:
- added C13: 10u, Capacitor_SMD:C_0603_1608Metric, symbol Device:C_Small
- added C14, C15: 100n, Capacitor_SMD:C_0603_1608Metric, symbol Device:C_Small
Connections:
- net +3V3: now also C13.2, C14.2, C15.2
- net GND: now also C13.1, C14.1, C15.1
Other:
- moved on the sheet: C11, C12, D2, R13

Commit message: fixes
Parts:
- R9: value 10K -> 1K
Connections:
- net at D1.1 (K): now also Q1.3 (C); no longer R2.2
- net at D1.2 (A): now also R2.2; no longer Q1.3 (C)
Other:
- moved on the sheet: D1
Changed lines of the file:
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@@
     (pin "1")
   )
-  (symbol (lib_id "LED:TSAL4400") (at 204.47 74.93 270) (unit 1)
-    (in_bom yes) (on_board yes) (fields_autoplaced)
-    (property "Reference" "D1" (id 0) (at 208.28 72.5169 90)
-      (effects (font (size 1.27 1.27)) (justify left))
-    )
-    (property "Value" "TSAL6200" (id 1) (at 208.28 75.0569 90)
-      (effects (font (size 1.27 1.27)) (justify left))
-    )
-    (property "Footprint" "LED_THT:LED_D3.0mm_IRBlack" (id 2) (at 208.915 74.93 0)
+  (symbol (lib_id "LED:TSAL4400") (at 204.47 72.39 90) (unit 1)
+    (in_bom yes) (on_board yes) (fields_autoplaced)
+    (property "Reference" "D1" (id 0) (at 207.01 72.2629 90)
+      (effects (font (size 1.27 1.27)) (justify right))
+    )
+    (property "Value" "TSAL6200" (id 1) (at 207.01 74.8029 90)
+      (effects (font (size 1.27 1.27)) (justify right))
+    )
+    (property "Footprint" "LED_THT:LED_D3.0mm_IRBlack" (id 2) (at 200.025 72.39 0)
       (effects (font (size 1.27 1.27)) hide)
     )
@@
     (in_bom yes) (on_board yes) (fields_autoplaced)
     (property "Reference" "R9" (id 0) (at 263.525 100.33 90))
-    (property "Value" "10K" (id 1) (at 263.525 102.87 90))
+    (property "Value" "1K" (id 1) (at 263.525 102.87 90))
     (property "Footprint" "Resistor_SMD:R_0603_1608Metric" (id 2) (at 263.525 106.68 0)
       (effects (font (size 1.27 1.27)) hide)
@@
     )
     (path "/c030f569-41ca-40ed-b543-9f41c1c76c1e"
-      (reference "R9") (unit 1) (value "10K") (footprint "Resistor_SMD:R_0603_1608Metric")
+      (reference "R9") (unit 1) (value "1K") (footprint "Resistor_SMD:R_0603_1608Metric")
     )
     (path "/1cadfc47-f42d-445e-a6e7-32c4fdd5bfca"
